Commit message: Changes to work with boris at bham

File: lwr_description/model/kuka_lwr.urdf.xacro (robot description, xacro)
@@ -31,5 +31,5 @@
 				<mass value="${base_mass}"/>
 				<origin xyz="0 0 0.055"  />
-				<cylinder_inertia_def radius="0.06" length="0.11" mass="${base_mass}"/>
+				<xacro:cylinder_inertia_def radius="0.06" length="0.11" mass="${base_mass}"/>
 			</inertial>
 			<visual>
@@ -38,5 +38,5 @@
 					<mesh filename="package://lwr_description/meshes/lwr4plus/visual/base.STL"/>
 				</geometry>
-				<material name="Kuka/Orange"/>
+				<material name="Kuka/Blue"/>
 			</visual>
 			<collision>
@@ -68,5 +68,5 @@
 				<mass value="${link_mass}"/>
 				<origin rpy="0 0 0" xyz="0 -0.06 0.130"/>
-				<cuboid_inertia_def length="0.12" width="0.06" height="0.260" mass="${link_mass}"/>
+				<xacro:cuboid_inertia_def length="0.12" width="0.06" height="0.260" mass="${link_mass}"/>
 			</inertial>
 			<visual>
@@ -75,5 +75,5 @@
 					<mesh filename="package://lwr_description/meshes/lwr4plus/visual/link_1.STL"/>
 				</geometry>
-				<material name="Kuka/Orange"/>
+				<material name="Kuka/Blue"/>
 			</visual>
 			<collision>
@@ -117,5 +117,5 @@
 				<mass value="${link_mass}"/>
 				<origin rpy="0 0 0" xyz="0 0.06 ${0.130 - 0.06}"/>
-				<cuboid_inertia_def length="0.12" width="0.06" height="0.260" mass="${link_mass}"/>
+				<xacro:cuboid_inertia_def length="0.12" width="0.06" height="0.260" mass="${link_mass}"/>
 			</inertial>
 			<visual>
@@ -124,5 +124,5 @@
 					<mesh filename="package://lwr_description/meshes/lwr4plus/visual/link_2.STL"/>
 				</geometry>
-				<material name="Kuka/Orange"/>
+				<material name="Kuka/Blue"/>
 			</visual>
 			<collision>
@@ -166,5 +166,5 @@
 				<mass value="${link_mass}"/>
 				<origin rpy="0 0 0" xyz="0 0.06 0.130"/>
-				<cuboid_inertia_def length="0.12" width="0.06" height="0.260" mass="${link_mass}"/>
+				<xacro:cuboid_inertia_def length="0.12" width="0.06" height="0.260" mass="${link_mass}"/>
 			</inertial>
 			<visual>
@@ -173,5 +173,5 @@
 					<mesh filename="package://lwr_description/meshes/lwr4plus/visual/link_3.STL"/>
 				</geometry>
-				<material name="Kuka/Orange"/>
+				<material name="Kuka/Blue"/>
 			</visual>
 			<collision>
@@ -215,5 +215,5 @@
 				<mass value="${link_mass}"/>
 				<origin rpy="0 0 0" xyz="0 -0.06 ${0.130 - 0.06}"/>
-				<cuboid_inertia_def length="0.12" width="0.06" height="0.2600" mass="${link_mass}"/>
+				<xacro:cuboid_inertia_def length="0.12" width="0.06" height="0.2600" mass="${link_mass}"/>
 			</inertial>
 			<visual>
@@ -222,5 +222,5 @@
 					<mesh filename="package://lwr_description/meshes/lwr4plus/visual/link_4.STL"/>
 				</geometry>
-				<material name="Kuka/Orange"/>
+				<material name="Kuka/Blue"/>
 			</visual>
 			<collision>
@@ -264,5 +264,5 @@
 				<mass value="${link_mass}"/>
 				<origin rpy="0 0 0" xyz="0 0 0.124"/>
-				<cuboid_inertia_def length="0.12" width="0.06" height="0.248" mass="${link_mass}"/>
+				<xacro:cuboid_inertia_def length="0.12" width="0.06" height="0.248" mass="${link_mass}"/>
 			</inertial>
 			<visual>
@@ -271,5 +271,5 @@
 					<mesh filename="package://lwr_description/meshes/lwr4plus/visual/link_5.STL"/>
 				</geometry>
-				<material name="Kuka/Orange"/>
+				<material name="Kuka/Blue"/>
 			</visual>
 			<collision>
@@ -313,5 +313,5 @@
 				<mass value="${wrist_mass}"/>
 				<origin rpy="0 0 0" xyz="0 0 0.0625"/>
-				<cuboid_inertia_def length="0.125" width="0.125" height="0.125" mass="${wrist_mass}"/>
+				<xacro:cuboid_inertia_def length="0.125" width="0.125" height="0.125" mass="${wrist_mass}"/>
 			</inertial>
 			<visual>
@@ -350,5 +350,5 @@
 				<mass value="${tip_mass}"/>
 				<origin xyz="0 0 0"/>
-				<cuboid_inertia_def length="0.1" width="0.1" height="0.1" mass="${tip_mass}"/>
+				<xacro:cuboid_inertia_def length="0.1" width="0.1" height="0.1" mass="${tip_mass}"/>
 			</inertial>
 			<visual>

File: lwr_description/model/kuka_materials.xacro (robot description, xacro)
@@ -23,5 +23,5 @@
   </material>
   <material name="Kuka/Blue">
-    <color rgba="0.0 0.0 0.8 1.0"/>
+    <color rgba="0.1 0.4 0.6 1.0"/>
   </material>
 </robot>
